File: rsc/schematics/NPN Switch/NPN Switch.sch (KiCad schematic (older format))
At the start: 3 parts, among them Q1 Q_NPN_CBE

Commit message: kicad v0.1 first pass generation pdf from kicad schematics still fail one sheet generation
Connections:
- net labels added: VIN, VOUT
- net labels removed: IN
- wire segments 8 -> 10
Changed lines of the file:
@@
 U 1 1 5EC35F6C
 P 6000 2700
-F 0 "LOAD" H 6070 2746 50  0000 L CNN
+F 0 "LOAD" V 5900 2600 50  0000 L CNN
 F 1 "R" H 6070 2655 50  0001 L CNN
 F 2 "" V 5930 2700 50  0001 C CNN
@@
 	5550 3150 5700 3150
 Wire Wire Line
-	6000 2850 6000 2950
+	6000 2850 6000 2900
 Wire Wire Line
 	6000 2500 6000 2550
@@
 	5000 3150 5250 3150
 Text Label 5000 3150 0    50   ~ 0
-IN
+VIN
 Wire Wire Line
 	5000 2950 5200 2950
@@
 Wire Wire Line
 	6000 3350 6000 3450
+Wire Wire Line
+	6000 2900 6250 2900
+Connection ~ 6000 2900
+Wire Wire Line
+	6000 2900 6000 2950
+Text Label 6100 2900 0    50   ~ 0
+VOUT
 $EndSCHEMATC
