File: rsc/schematics/cmos inverter/cmos inverter.sch (KiCad schematic (older format))
At the start: 3 parts, among them Q1 Q_PMOS_GDS, Q2 Q_NMOS_SGD

Commit message: kicad_v0.2a adding backlog of DP
Connections:
- net labels added: VIN, VOUT
- net labels removed: IN, OUT
Changed lines of the file:
@@
 EESchema Schematic File Version 4
+LIBS:cmos inverter-cache
 EELAYER 30 0
 EELAYER END
@@
 	5950 2700 5950 2800
 Text Label 6200 2700 0    50   ~ 0
-OUT
+VOUT
 Text Label 5350 2700 0    50   ~ 0
-IN
+VIN
 $Comp
 L power:GND #PWR?
